Commit message: Syncing work

File: oro_v4/urdf/oro_v4.urdf (robot description, URDF)
Before this commit: robot oro_v4, 8 links, 7 joints
Links:
- removed link wheel_left
- removed link wheel_right
- added link base_footprint
- added link caster_back_left_link, mass 0.005; collision box size=0.030 0.009 0.020
- added link caster_back_right_link, mass 0.005; collision box size=0.030 0.009 0.020
- added link imu_link
- added link wheel_left_link, mass 2.8498940e-02; collision cylinder length=0.018 radius=0.033; visual mesh filename=package://oro_description/meshes/wheels/left_tire.stl scale=0.001 0.001 0.001
- added link wheel_right_link, mass 2.8498940e-02; collision cylinder length=0.018 radius=0.033; visual mesh filename=package://oro_description/meshes/wheels/right_tire.stl scale=0.001 0.001 0.001
- link base_link: mass 1.32433600289921 -> 1.3729096e+00; geometry collision box size=0.266 0.266 0.094; visual mesh filename=package://oro_description/meshes/bases/waffle_base.stl scale=0.001 0.001 0.001
Joints:
- added joint base_joint: type fixed, parent base_footprint, child base_link, origin xyz=0 0 0.010 rpy=0 0 0
- added joint caster_back_left_joint: type fixed, parent base_link, child caster_back_left_link, origin xyz=-0.177 0.064 -0.004 rpy=-1.57 0 0
- added joint caster_back_right_joint: type fixed, parent base_link, child caster_back_right_link, origin xyz=-0.177 -0.064 -0.004 rpy=-1.57 0 0
- added joint imu_joint: type fixed, parent base_link, child imu_link, origin xyz=0.0 0 0.068 rpy=0 0 0
- added joint scan_joint: type fixed, parent base_link, child base_scan, origin xyz=-0.064 0 0.122 rpy=0 0 0
- joint neck_joint: origin xyz=-0.111522868965688 -0.223111765630108 0.978912848528942 rpy=0 0 -0.00709484089756157 -> xyz=-0.111522868965688 -0.223111765630108 1.00151376852 rpy=0 0 0
- joint wheel_left_joint: axis 0 1 0 -> 0 0 1; child wheel_left -> wheel_left_link; origin xyz=-0.242519526797119 -0.170162162680993 -0.018480323531233 rpy=0 0.149555140664513 3.13449781269223 -> xyz=0.0 0.144 0.023 rpy=-1.57 0 0
- joint wheel_right_joint: axis 0 1 0 -> 0 0 1; child wheel_right -> wheel_right_link; origin xyz=-0.24060539870727 0.0996248558539564 -0.018480323531233 rpy=0 -0.444631589877229 -0.00709484089756432 -> xyz=0.0 -0.144 0.023 rpy=-1.57 0 0
