Commit message: Migrating urdf to new version

File: oro_description_new/urdf/oro_description.urdf (robot description, URDF)
Before this commit: robot oro_description, 8 links, 7 joints
Links:
- removed link wheel_left
- removed link wheel_right
- added link base_footprint
- added link caster_back_left_link, mass 0.005; collision box size=0.030 0.009 0.020
- added link caster_back_right_link, mass 0.005; collision box size=0.030 0.009 0.020
- added link wheel_left_link, mass 2.8498940e-02; collision cylinder length=0.018 radius=0.033; visual mesh filename=package://oro_description/meshes/wheels/left_tire.stl scale=0.001 0.001 0.001
- added link wheel_right_link, mass 2.8498940e-02; collision cylinder length=0.018 radius=0.033; visual mesh filename=package://oro_description/meshes/wheels/right_tire.stl scale=0.001 0.001 0.001
- link base_link: mass 1.32433599991547 -> 1.3729096e+00; geometry collision box size=0.266 0.266 0.094; visual mesh filename=package://oro_description/meshes/base_link.STL
Joints:
- added joint base_joint: type fixed, parent base_footprint, child base_link, origin xyz=0 0 0.010 rpy=0 0 0
- added joint caster_back_left_joint: type fixed, parent base_link, child caster_back_left_link, origin xyz=-0.177 0.064 -0.004 rpy=-1.57 0 0
- added joint caster_back_right_joint: type fixed, parent base_link, child caster_back_right_link, origin xyz=-0.177 -0.064 -0.004 rpy=-1.57 0 0
- joint wheel_left_joint: axis 0 1 0 -> 0 0 1; child wheel_left -> wheel_left_link; origin xyz=-0.242519526797119 -0.170162162680993 -0.018480323531233 rpy=0 0.149555140664513 3.13449781269223 -> xyz=0.0 0.144 0.023 rpy=-1.57 0 0
- joint wheel_right_joint: axis 0 1 0 -> 0 0 1; child wheel_right -> wheel_right_link; origin xyz=-0.24060539870727 0.0996248558539564 -0.018480323531233 rpy=0 -0.444631589877229 -0.00709484089756432 -> xyz=0.0 -0.144 0.023 rpy=-1.57 0 0

Commit message: Adding another new version

File: oro_description_new/urdf/oro_description.urdf (robot description, URDF)
Before this commit: robot oro, 11 links, 10 joints
Links:
- link base_link: geometry collision box size=0.266 0.266 0.094; visual mesh filename=package://oro_description/meshes/bases/waffle_base.stl scale=0.001 0.001 0.001
- link base_scan: mass 0.0530538693608539 -> 0.0530538307331328
- link depth_cam: mass 0.153126622817504 -> 0.153126622909889
- link neck: mass 1.109267558899 -> 1.10926755879378
- link pan: mass 0.0446711230149848 -> 0.0446711336598691
- link tilt: mass 0.190333592774622 -> 0.190333563757372
Joints:
- joint base_scan_joint: origin xyz=-0.29299616822181 -0.034903733333453 0.069469676468767 rpy=1.5707963267949 0 -0.00709484089756434 -> xyz=-0.293 -0.034904 0.06947 rpy=0 0 0
- joint depth_cam_joint: origin xyz=0.087462 0 0 rpy=-1.5708 0 0 -> xyz=0.0874623622012928 0 0 rpy=-1.57079632679489 0 0
- joint neck_joint: origin xyz=-0.111522868965688 -0.223111765630108 0.978912848528942 rpy=0 0 -0.00709484089756157 -> xyz=-0.111522868965688 -0.223111765630108 0.978912848528942 rpy=0 0 0
- joint pan_joint: origin xyz=-0.080369 0.18689 0.049257 rpy=0 0 -0.0075711 -> xyz=-0.0803690267279755 0.186890382040786 0.0492568279398251 rpy=0 0 -0.00757105682660417
- joint tilt_joint: origin xyz=0.00025 0 0.04208 rpy=-3.127 0 -1.5708 -> xyz=0.000250000000001249 0 0.0420800000000014 rpy=-3.12696731241166 0 -1.5707963267949

Commit message: Syncing workspaces

File: oro_description_new/urdf/oro_description.urdf (robot description, URDF)
Before this commit: robot oro, 11 links, 10 joints
Links:
- link base_link: geometry collision box size=0.266 0.266 0.094; visual mesh filename=package://oro_description/meshes/bases/waffle_base.stl scale=0.001 0.001 0.001
