Commit message: Syncing

File: oro_v6/urdf/oro.gazebo.xacro (robot description, xacro)
@@ -53,7 +53,10 @@
   </gazebo>
   <!--TODO: Ensure that this is working-->
-  <gazebo>
-    <plugin name="gazebo_ros_control" filename="libgazebo_ros_control.so"/>
-  </gazebo>
+    <gazebo>
+        <plugin name="gazebo_ros_control" filename="libgazebo_ros_control.so">
+            <robotNamespace>/</robotNamespace>
+	    <robotSimType>gazebo_ros_control/DefaultRobotHWSim</robotSimType>
+        </plugin>
+    </gazebo>
   <gazebo>
     <plugin name="oro_diff_controller" filename="libgazebo_ros_diff_drive.so">

File: oro_v6/urdf/oro.transmission.xacro (robot description, xacro)
@@ -4,8 +4,8 @@
     <type>transmission_interface/SimpleTransmission</type>
     <joint name="pan_joint">
-      <hardwareInterface>EffortJointInterface</hardwareInterface>
+	    <hardwareInterface>hardware_interface/EffortJointInterface</hardwareInterface>
     </joint>
     <actuator name="pan_dynamixel">
-      <hardwareInterface>EffortJointInterface</hardwareInterface>
+	    <hardwareInterface>hardware_interface/EffortJointInterface</hardwareInterface>
       <mechanicalReduction>1</mechanicalReduction>
     </actuator>
@@ -14,8 +14,8 @@
     <type>transmission_interface/SimpleTransmission</type>
     <joint name="tilt_joint">
-      <hardwareInterface>EffortJointInterface</hardwareInterface>
+      <hardwareInterface>hardware_interface/EffortJointInterface</hardwareInterface>
     </joint>
     <actuator name="tilt_dynamixel">
-      <hardwareInterface>EffortJointInterface</hardwareInterface>
+	    <hardwareInterface>hardware_interface/EffortJointInterface</hardwareInterface>
       <mechanicalReduction>1</mechanicalReduction>
     </actuator>

File: oro_v6/urdf/oro_v6.urdf (robot description, URDF)
Before this commit: robot oro, 12 links, 11 joints
Joints:
- joint depth_cam_joint: type continuous -> fixed
