Commit message: Fixed gazebo simulation

File: oro_v6/urdf/oro_v6.xacro (robot description, xacro)
@@ -2,6 +2,6 @@
 <!--Author: Thomas Herring-->
 <robot name="oro" xmlns:xacro="http://ros.org/wiki/xacro">
+    <xacro:include filename="$(find oro_v6)/urdf/oro.gazebo" />
     <xacro:include filename="$(find oro_v6)/urdf/common_properties.xacro" />
-    <xacro:include filename="$(find oro_v6)/urdf/oro.gazebo.xacro" />
     <link name="base_footprint" />
     <link name="base_link">
@@ -71,5 +71,5 @@
             <origin xyz="-2.50155840103294E-05 -3.07858331118488E-05 0.0205898386906647" rpy="0 0 0" />
             <mass value="0.0446711229185335" />
-            <inertia ixx="1.24180241554179E-05" ixy="-4.29119054419149E-13" ixz="2.4476376713091E-09" iyy="1.04151202907413E-05" iyz="-1.82749851584174E-07" izz="7.78082243124466E-06" />
+            <inertia ixx="0" ixy="0" ixz="0" iyy="0" iyz="0" izz="0" />
         </inertial>
         <visual>
@@ -99,5 +99,6 @@
             <origin xyz="0.00118385527699938 0.0139616359862273 -0.0783421837132381" rpy="0 0 0" />
             <mass value="0.190333592129278" />
-            <inertia ixx="0.000184137194903989" ixy="-1.52842480239196E-06" ixz="6.62804385986339E-08" iyy="0.000483856390372872" iyz="5.06450642269179E-08" izz="0.000309913696954649" />
+            <!--<inertia ixx="0.000184137194903989" ixy="-1.52842480239196E-06" ixz="6.62804385986339E-08" iyy="0.000483856390372872" iyz="5.06450642269179E-08" izz="0.000309913696954649" />-->
+            <inertia ixx="0" ixy="0" ixz="0" iyy="0" iyz="0" izz="0" />
         </inertial>
         <visual>
@@ -127,5 +128,6 @@
             <origin xyz="1.57606088716095E-05 4.46446457198904E-10 4.41076423673969E-06" rpy="0 0 0" />
             <mass value="0.153126621719673" />
-            <inertia ixx="0.000375847392851875" ixy="1.29137498226285E-13" ixz="-2.267576442511E-09" iyy="2.29360924151489E-05" iyz="1.98626115179079E-12" izz="0.000377927282615239" />
+            <!--<inertia ixx="0.000375847392851875" ixy="1.29137498226285E-13" ixz="-2.267576442511E-09" iyy="2.29360924151489E-05" iyz="1.98626115179079E-12" izz="0.000377927282615239" />-->
+            <inertia ixx="0" ixy="0" ixz="0" iyy="0" iyz="0" izz="0" />
         </inertial>
         <visual>
@@ -321,24 +323,24 @@
         <!--</actuator>-->
     <!--</transmission>-->
-    <!--<transmission name="trans_wheel_right_joint">-->
-        <!--<type>transmission_interface/SimpleTransmission</type>-->
-        <!--<joint name="wheel_right_joint">-->
-            <!--<hardwareInterface>hardware_interface/EffortJointInterface</hardwareInterface>-->
-        <!--</joint>-->
-        <!--<actuator name="wheel_right_joint_motor">-->
-            <!--<hardwareInterface>hardware_interface/EffortJointInterface</hardwareInterface>-->
-            <!--<mechanicalReduction>1</mechanicalReduction>-->
-        <!--</actuator>-->
-    <!--</transmission>-->
-    <!--<transmission name="trans_wheel_left_joint">-->
-        <!--<type>transmission_interface/SimpleTransmission</type>-->
-        <!--<joint name="wheel_left_joint">-->
-            <!--<hardwareInterface>hardware_interface/EffortJointInterface</hardwareInterface>-->
-        <!--</joint>-->
-        <!--<actuator name="wheel_left_joint_motor">-->
-            <!--<hardwareInterface>hardware_interface/EffortJointInterface</hardwareInterface>-->
-            <!--<mechanicalReduction>1</mechanicalReduction>-->
-        <!--</actuator>-->
-    <!--</transmission>-->
+    <transmission name="trans_wheel_right_joint">
+	<type>transmission_interface/SimpleTransmission</type>
+	<joint name="wheel_right_joint">
+	    <hardwareInterface>hardware_interface/EffortJointInterface</hardwareInterface>
+	</joint>
+	<actuator name="wheel_right_joint_motor">
+	    <hardwareInterface>hardware_interface/EffortJointInterface</hardwareInterface>
+	    <mechanicalReduction>1</mechanicalReduction>
+	</actuator>
+    </transmission>
+    <transmission name="trans_wheel_left_joint">
+	<type>transmission_interface/SimpleTransmission</type>
+	<joint name="wheel_left_joint">
+	    <hardwareInterface>hardware_interface/EffortJointInterface</hardwareInterface>
+	</joint>
+	<actuator name="wheel_left_joint_motor">
+	    <hardwareInterface>hardware_interface/EffortJointInterface</hardwareInterface>
+	    <mechanicalReduction>1</mechanicalReduction>
+	</actuator>
+    </transmission>
     <gazebo>
         <plugin name="gazebo_ros_control" filename="libgazebo_ros_control.so">

Commit message: Added inertia changes

File: oro_v6/urdf/oro_v6.xacro (robot description, xacro)
@@ -99,6 +99,6 @@
             <origin xyz="0.00118385527699938 0.0139616359862273 -0.0783421837132381" rpy="0 0 0" />
             <mass value="0.190333592129278" />
-            <!--<inertia ixx="0.000184137194903989" ixy="-1.52842480239196E-06" ixz="6.62804385986339E-08" iyy="0.000483856390372872" iyz="5.06450642269179E-08" izz="0.000309913696954649" />-->
-            <inertia ixx="0" ixy="0" ixz="0" iyy="0" iyz="0" izz="0" />
+	    <inertia ixx="0.000184137194903989" ixy="-1.52842480239196E-06" ixz="6.62804385986339E-08" iyy="0.000483856390372872" iyz="5.06450642269179E-08" izz="0.000309913696954649" />
+            <!--<inertia ixx="0" ixy="0" ixz="0" iyy="0" iyz="0" izz="0" />-->
         </inertial>
         <visual>

Commit message: Modified controller startup

File: oro_v6/urdf/oro_v6.xacro (robot description, xacro)
@@ -22,8 +22,18 @@
             </geometry>
         </collision>
-<inertial>
-            <mass value="4" />
-            <inertia ixx="0.03" iyy="0.03" izz="0.03" ixy="0.0" ixz="0.0" iyz="0.0" />
-        </inertial>
+    <inertial>
+      <origin
+        xyz="-0.059236 -0.00035128 0.020158"
+        rpy="0 0 0" />
+      <mass
+        value="1.3214" />
+      <inertia
+        ixx="0.0013555"
+        ixy="-1.9279E-07"
+        ixz="5.0224E-08"
+        iyy="0.00061741"
+        iyz="1.2847E-06"
+        izz="0.0019406" />
+    </inertial>
     </link>
     <joint name="base_joint" type="fixed">
@@ -40,9 +50,18 @@
     <link name="imu_link" />
     <link name="neck">
-<inertial>
-            <origin xyz="5.1035235981059E-05 3.02250471614812E-06 0.451367324075199" rpy="0 0 0" />
-            <mass value="1.10926754952808" />
-            <inertia ixx="0.0564255773084723" ixy="-9.03977213539269E-10" ixz="-1.82951888591032E-07" iyy="0.0564818854150741" iyz="-4.18069407423454E-11" izz="0.000391068830002547" />
-        </inertial>
+    <inertial>
+      <origin
+        xyz="5.10352359810728E-05 3.02250471614803E-06 0.451367324075199"
+        rpy="0 0 0" />
+      <mass
+        value="1.10926754952808" />
+      <inertia
+        ixx="0.0564255773084723"
+        ixy="-9.03977213538345E-10"
+        ixz="-1.82951888591033E-07"
+        iyy="0.0564818854150741"
+        iyz="-4.18069407410363E-11"
+        izz="0.000391068830002547" />
+    </inertial>
         <visual>
             <origin xyz="0 0 0" rpy="0 0 0" />
@@ -68,9 +87,18 @@
     </joint>
     <link name="pan">
-<inertial>
-            <origin xyz="-2.50155840103294E-05 -3.07858331118488E-05 0.0205898386906647" rpy="0 0 0" />
-            <mass value="0.0446711229185335" />
-            <inertia ixx="0" ixy="0" ixz="0" iyy="0" iyz="0" izz="0" />
-        </inertial>
+    <inertial>
+      <origin
+        xyz="-2.50155840103225E-05 -3.0785833111849E-05 0.0205898386906644"
+        rpy="0 0 0" />
+      <mass
+        value="0.0446711229185335" />
+      <inertia
+        ixx="1.24180241554179E-05"
+        ixy="-4.29119054508693E-13"
+        ixz="2.44763767130923E-09"
+        iyy="1.04151202907413E-05"
+        iyz="-1.82749851584174E-07"
+        izz="7.78082243124466E-06" />
+    </inertial>
         <visual>
             <origin xyz="0 0 0" rpy="0 0 0" />
@@ -96,10 +124,18 @@
     </joint>
     <link name="tilt">
-<inertial>
-            <origin xyz="0.00118385527699938 0.0139616359862273 -0.0783421837132381" rpy="0 0 0" />
-            <mass value="0.190333592129278" />
-	    <inertia ixx="0.000184137194903989" ixy="-1.52842480239196E-06" ixz="6.62804385986339E-08" iyy="0.000483856390372872" iyz="5.06450642269179E-08" izz="0.000309913696954649" />
-            <!--<inertia ixx="0" ixy="0" ixz="0" iyy="0" iyz="0" izz="0" />-->
-        </inertial>
+    <inertial>
+      <origin
+        xyz="0.00118385527699939 0.0139616359862273 -0.0783421837132381"
+        rpy="0 0 0" />
+      <mass
+        value="0.190333592129278" />
+      <inertia
+        ixx="0.000184137194903989"
+        ixy="-1.52842480239196E-06"
+        ixz="6.62804385986578E-08"
+        iyy="0.000483856390372872"
+        iyz="5.06450642269202E-08"
+        izz="0.000309913696954649" />
+    </inertial>
         <visual>
             <origin xyz="0 0 0" rpy="0 0 0" />
@@ -125,10 +161,18 @@
     </joint>
     <link name="depth_cam">
-<inertial>
-            <origin xyz="1.57606088716095E-05 4.46446457198904E-10 4.41076423673969E-06" rpy="0 0 0" />
-            <mass value="0.153126621719673" />
-            <!--<inertia ixx="0.000375847392851875" ixy="1.29137498226285E-13" ixz="-2.267576442511E-09" iyy="2.29360924151489E-05" iyz="1.98626115179079E-12" izz="0.000377927282615239" />-->
-            <inertia ixx="0" ixy="0" ixz="0" iyy="0" iyz="0" izz="0" />
-        </inertial>
+    <inertial>
+      <origin
+        xyz="1.5761E-05 4.4645E-10 4.4108E-06"
+        rpy="0 0 0" />
+      <mass
+        value="0.15313" />
+      <inertia
+        ixx="0.00037585"
+        ixy="1.2914E-13"
+        ixz="-2.2676E-09"
+        iyy="2.2936E-05"
+        iyz="1.9863E-12"
+        izz="0.00037793" />
+    </inertial>
         <visual>
             <origin xyz="0 0 0" rpy="0 0 0" />
@@ -154,9 +198,18 @@
     </joint>
     <link name="base_scan">
-<inertial>
-            <origin xyz="-0.00862865863959542 -1.73967868891126E-05 0.000140843030897758" rpy="0 0 0" />
-            <mass value="0.0530538694104072" />
-            <inertia ixx="1.81416003681575E-05" ixy="2.62458054720209E-08" ixz="-4.99055692614565E-06" iyy="3.57220957812171E-05" iyz="1.92490809961403E-08" izz="4.4601102506138E-05" />
-        </inertial>
+    <inertial>
+      <origin
+        xyz="-0.00862865863959544 -1.73967868891075E-05 0.000140843030897758"
+        rpy="0 0 0" />
+      <mass
+        value="0.0530538694104072" />
+      <inertia
+        ixx="1.81416003681575E-05"
+        ixy="2.62458054720224E-08"
+        ixz="-4.99055692614564E-06"
+        iyy="3.57220957812171E-05"
+        iyz="1.92490809961388E-08"
+        izz="4.46011025061381E-05" />
+    </inertial>
         <visual>
             <origin xyz="0 0 0" rpy="0 0 0" />
